File: pcb/CurrentVoltage_Sensor.kicad_pcb (KiCad board)
At the start: 2 copper layers, 34.5 x 26 mm, 13 parts, among them J1 Wago_734-164_1x04_P3.50mm

Commit message: PCB update
Parts:
- R1: value LRMAP3920C-R0015FT -> HoLRS1575-1.5mR-1%
- moved H1 1.00 mm to (109.5, 85.0)
- moved H5 1.00 mm to (109.5, 101.0)
- moved H2 0.50 mm to (135.5, 85.0)
- moved H6 0.50 mm to (135.5, 101.0)
- moved R1 0.50 mm to (122.0, 85.0)
- moved REF** 0.50 mm to (126.5, 90.5)
- moved ADR0 0.21 mm to (110.8, 96.1)
- moved ADR1 0.20 mm to (110.8, 92.0)
- moved LTC4151 0.20 mm to (123.0, 91.0)
Routing:
- net +BATT: track 14.0 -> 0.00 mm, vias 24 -> 10
- net /Sense_{+}: track 5.48 -> 7.18 mm
- net /V_{out}: vias 25 -> 11
Other:
- board size 34.5 x 26 mm -> 36 x 26 mm

Commit message: PCB v1.1 - Fixed some PCB traces
Routing:
- net +BATT: track 0.00 -> 17.5 mm
Other:
- board text added: "VI Sensor v1.1 V_{IN} = 7V - 80V I_{meas, max} = 54A"
- board text removed: "VI Sensor v1.0 V_{IN} = 7V - 80V I_{meas, max} = 54A"
Changed lines of the file:
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@@
     (property "ki_keywords" "Solder Jumper SPDT")
     (attr exclude_from_pos_files)
-    (fp_text reference "ADR0" (at 4.8 0.07 180) (layer "B.SilkS")
+    (fp_text reference "ADR0" (at 4.8 0.07) (layer "B.SilkS")
         (effects (font (size 0.8 0.8) (thickness 0.15)) (justify mirror))
     )
@@
         (effects (font (size 1 1) (thickness 0.15)) (justify mirror))
     )
-    (fp_text user "L" (at 2.3 2.07 180) (layer "B.SilkS")
+    (fp_text user "L" (at 2.3 2.07) (layer "B.SilkS")
         (effects (font (size 1 1) (thickness 0.15)) (justify mirror))
     )
-    (fp_text user "H" (at -2.2 2.07 180) (layer "B.SilkS")
+    (fp_text user "H" (at -2.2 2.07) (layer "B.SilkS")
         (effects (font (size 1 1) (thickness 0.15)) (justify mirror))
     )
@@
     (fp_line (start 3 -1.25) (end 3 1.27)
       (stroke (width 0.05) (type solid)) (layer "B.CrtYd"))
-    (pad "" smd rect (at -1.2 0 180) (size 1.5 1.5) (layers "B.Mask"))
-    (pad "" smd rect (at 1.2 0 180) (size 1.5 1.5) (layers "B.Mask"))
+    (pad "" smd rect (at -1.475 0 180) (size 2.05 1.5) (layers "B.Mask"))
+    (pad "" smd rect (at 1.025 0 180) (size 2.95 1.5) (layers "B.Mask"))
     (pad "1" smd custom (at -2 0 180) (size 0.3 0.3) (layers "B.Cu" "B.Mask")
       (net 1 "+BATT") (pinfunction "A") (pintype "passive") (zone_connect 2)
@@
     (fp_line (start 3 -1.25) (end 3 1.27)
       (stroke (width 0.05) (type solid)) (layer "B.CrtYd"))
-    (pad "" smd rect (at -1.2 0 180) (size 1.5 1.5) (layers "B.Mask"))
-    (pad "" smd rect (at 1.2 0 180) (size 1.5 1.5) (layers "B.Mask"))
+    (pad "" smd rect (at -1.25 0 180) (size 2.5 1.5) (layers "B.Mask"))
+    (pad "" smd rect (at 1.25 0 180) (size 2.5 1.5) (layers "B.Mask"))
     (pad "1" smd custom (at -2 0 180) (size 0.3 0.3) (layers "B.Cu" "B.Mask")
       (net 1 "+BATT") (pinfunction "A") (pintype "passive") (zone_connect 2)
@@
     (effects (font (size 0.8 0.8) (thickness 0.15)) (justify bottom mirror))
   )
-  (gr_text "VI Sensor v1.0\nV_{IN} = 7V - 80V\nI_{meas, max} = 54A" (at 129 86) (layer "B.SilkS")
+  (gr_text "VI Sensor v1.1\nV_{IN} = 7V - 80V\nI_{meas, max} = 54A" (at 129 86) (layer "B.SilkS")
     (effects (font (size 1 1) (thickness 0.15)) (justify left bottom mirror))
   )
@@
     (effects (font (size 2 2) (thickness 0.15)) (justify left bottom))
   )
+  (segment (start 115 85.50962) (end 119.99038 90.5) (width 0.25) (layer "F.Cu") (net 1))
+  (segment (start 115 84.5) (end 115 85.50962) (width 0.25) (layer "F.Cu") (net 1))
+  (segment (start 119.99038 90.5) (end 120.8 90.5) (width 0.25) (layer "F.Cu") (net 1))
   (via (at 105.5 85.5) (size 0.8) (drill 0.4) (layers "F.Cu" "B.Cu") (free) (net 1))
   (via (at 112.5 88) (size 0.8) (drill 0.4) (layers "F.Cu" "B.Cu") (free) (net 1))
@@
   (via (at 108 81) (size 0.8) (drill 0.4) (layers "F.Cu" "B.Cu") (free) (net 1))
   (via (at 106.5 82) (size 0.8) (drill 0.4) (layers "F.Cu" "B.Cu") (free) (net 1))
+  (segment (start 113.3 91.5) (end 113.3 88.8) (width 0.25) (layer "B.Cu") (net 1))
+  (segment (start 112.8 92) (end 113.3 91.5) (width 0.25) (layer "B.Cu") (net 1))
+  (segment (start 113.3 88.8) (end 112.5 88) (width 0.25) (layer "B.Cu") (net 1))
+  (segment (start 112.8 92) (end 112.8 96.07) (width 0.25) (layer "B.Cu") (net 1))
   (via (at 132.5 81) (size 0.8) (drill 0.4) (layers "F.Cu" "B.Cu") (free) (net 2))
   (via (at 139 88) (size 0.8) (drill 0.4) (layers "F.Cu" "B.Cu") (free) (net 2))
@@
   (segment (start 111 100.5) (end 110.5 101) (width 0.5) (layer "B.Cu") (net 4))
   (segment (start 109 99.5) (end 110.5 101) (width 0.5) (layer "B.Cu") (net 4))
-  (segment (start 113.5 91.5) (end 120.6 91.5) (width 0.3) (layer "F.Cu") (net 5))
-  (segment (start 111 94) (end 113.5 91.5) (width 0.3) (layer "F.Cu") (net 5))
+  (segment (start 111 94) (end 112.3225 94) (width 0.3) (layer "F.Cu") (net 5))
+  (segment (start 114.8225 91.5) (end 120.6 91.5) (width 0.3) (layer "F.Cu") (net 5))
+  (segment (start 112.3225 94) (end 114.8225 91.5) (width 0.3) (layer "F.Cu") (net 5))
   (via (at 111 94) (size 0.8) (drill 0.4) (layers "F.Cu" "B.Cu") (net 5))
   (segment (start 111 96) (end 111 94) (width 0.25) (layer "B.Cu") (net 5))
