File: pcb/CurrentVoltage_Sensor.kicad_sch (KiCad schematic)
At the start: 11 parts, among them J1 Wago_734-164_1x04_P3.50mm, U1 LTC4151xMS

Commit message: PCB v1.1 - Fixed some PCB traces
Parts:
- R1: value LRMAP3920C-R0015FT -> HoLRS1575-1.5mR-1%
Other:
- note added: "REVISIONS V 1.0 - First V 1.1 - Fixed PCB traces (PIN2 and solder jumper "H"s connected to V_{IN} now)"
Changed lines of the file:
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@@
     (stroke (width 0) (type default))
+  )
+  (text "REVISIONS\nV 1.0 - First\nV 1.1 - Fixed PCB traces (PIN2 and solder jumper \"H\"s connected to V_{IN} now)"
+    (at 27.94 179.705 0)
+    (effects (font (size 1.27 1.27)) (justify left bottom))
   )
   (text "V_{out}" (at 74.93 113.03 0)
@@
       (effects (font (size 1.27 1.27)) (justify right))
     )
-    (property "Value" "LRMAP3920C-R0015FT" (at 80.01 86.36 90)
+    (property "Value" "HoLRS1575-1.5mR-1%" (at 80.01 86.36 90)
       (effects (font (size 1.27 1.27)) (justify right))
     )
